File: glidepoint-uno.kicad_pcb (KiCad board)
At the start: 2 copper layers, 68.6 x 53.3 mm, 16 parts, among them J1 Power, J2 Digital/PWM, J3 Analog, J4 Digital/PWM, J5 Conn_01x12_Socket, SW1 SW_Push, SW2 SW_Push

Commit message: Add i2c pull-ups, switch to Alps tactile buttons.
Parts:
- added R2: 10k, Resistor_SMD:R_0805_2012Metric, B.Cu at (117.1, 57.0)
- added R3: 10k, Resistor_SMD:R_0805_2012Metric, B.Cu at (117.1, 55.1)
- added SW3: Right, buttons:SW_SKSTAAE010, F.Cu at (109.8, 87.4)
- SW1: value SW_Push -> Left; footprint mbk:Choc-1u -> buttons:SW_SKSTAAE010
- SW2: value SW_Push -> Middle; footprint mbk:Choc-1u -> buttons:SW_SKSTAAE010
- moved SW2 11.0 mm to (109.8, 73.4)
- moved SW1 3.00 mm to (109.8, 58.3)
Connections:
- J4 pad 6: /2 -> SW3
Routing:
- net SW3: track 0.00 -> 99.4 mm
- net +3V3: track 64.7 -> 93.5 mm
- net SCL: track 34.4 -> 56.7 mm
- net SW2: track 102.2 -> 113.3 mm, vias 1 -> 0
- net SDA: track 39.9 -> 42.7 mm
- net SW1: track 46.4 -> 48.5 mm, vias 1 -> 0
- net GND: vias 3 -> 4
